File: probe/kicad/garden-reporter-board.kicad_pcb (KiCad board)
At the start: 2 copper layers, 40.6 x 74.9 mm, 31 parts, among them J1 70543-0106, J2 Conn_01x02, J3 70543-0002, J4 70543-0002, J5 70543-0002, Q1 Q_NMOS_SGD, Q2 Q_PMOS_SGD, U1 MCP1700-3302E_TO92, U2 MCP1700-3302E_TO92, U3 MCP1700-1202E_TO92

Commit message: Route all
Parts:
- moved R5 17.5 mm to (170.9, 94.2)
- moved R4 7.91 mm to (162.3, 115.1), turned to 0 degrees
- moved C6 5.23 mm to (146.5, 119.9)
- moved J5 5.02 mm to (168.1, 102.1)
- moved U2 3.66 mm to (139.7, 120.7)
- moved C9 1.80 mm to (161.5, 100.1)
- moved U3 1.80 mm to (156.0, 99.0)
- moved C8 1.80 mm to (152.7, 98.1)
- moved C7 1.79 mm to (146.6, 124.0)
- moved J3 0.27 mm to (151.4, 121.7)
- moved J4 0.27 mm to (164.3, 121.7)
Routing:
- net /sensor_soil: track 0.00 -> 72.1 mm
- net VDD: track 0.00 -> 61.0 mm
- net /sensor_temp: track 0.00 -> 59.9 mm
- net /sensor_batt: track 0.00 -> 52.5 mm
- net +3.3V: track 0.00 -> 43.1 mm
- net +BATT: track 0.00 -> 41.8 mm
- net /sensor_light: track 0.00 -> 34.3 mm
- net /xbee_ON: track 0.00 -> 31.5 mm
- net Net-(J2-Pad2): track 0.00 -> 25.6 mm
- net Net-(R3-Pad1): track 0.00 -> 22.2 mm
- net Net-(J2-Pad1): track 0.00 -> 22.0 mm
- net +3.3VADC: track 0.00 -> 14.2 mm
- net +1V2: track 0.00 -> 11.0 mm
- net Net-(Q2-Pad2): track 0.00 -> 8.61 mm
Other:
- board text added: "xbee power"
- board text removed: "xbee p"

Commit message: Finish and verifiy routing, finish and verify BOM
Parts:
- moved J5 3.57 mm to (168.4, 105.7)
- moved C9 2.16 mm to (163.3, 101.3)
Routing:
- net +3.3VADC: track 14.2 -> 32.9 mm
- net /sensor_light: track 34.3 -> 37.7 mm
- net +1V2: track 11.0 -> 12.7 mm
